Commit message: Made code operational with basic bug fixes. Much more work to do.

File: Rpi_Python_Code/WM_Roboarm_Inv_Kin_Def.urdf (robot description, URDF)
Before this commit: robot WM-Roboarm, 5 links, 4 joints
Joints:
- joint elbow: limit lower=0.0 upper=0.548 effort=1000.0 velocity=0.5 -> lower=0.0 upper=3 effort=1000.0 velocity=0.5
- joint shoulder: limit lower=0.0 upper=0.548 effort=1000.0 velocity=0.5 -> lower=0.0 upper=3 effort=1000.0 velocity=0.5
- joint swivel: limit lower=0.785 upper=4.926 effort=1000.0 velocity=0.5 -> lower=0 upper=3 effort=1000.0 velocity=0.5
